File: Schema_init/DetecteurSonnore.brd (EAGLE design)
At the start: 67 x 36.8 mm, 13 parts, among them Q1 2N2222, Q2 2N2222

Commit message: Ajout chapter 2 Breadboard, chapter 3 Eagle
A continuer évidemment mais c’est un premier jet!
Connections:
- net N$11 renamed VDD
- net AGND: now also BUZZER.-
Changed lines of the file:
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@@
 <wire x1="31.4833" y1="28.194" x2="31.75" y2="27.94" width="0.5588" layer="16"/>
-</signal>
-<signal name="N$11">
-<contactref element="R2" pad="1"/>
-<contactref element="D3" pad="A"/>
-<wire x1="29.1338" y1="50.7492" x2="35.2425" y2="44.6405" width="0.5588" layer="16"/>
-<wire x1="35.2425" y1="44.6405" x2="35.56" y2="44.45" width="0.5588" layer="16"/>
-<wire x1="26.3144" y1="47.9298" x2="15.5067" y2="47.9298" width="0.5588" layer="16"/>
-<wire x1="29.1338" y1="50.7492" x2="26.3144" y2="47.9298" width="0.5588" layer="16"/>
-<wire x1="29.1338" y1="50.7492" x2="29.21" y2="50.8" width="0.5588" layer="16"/>
 </signal>
 <signal name="N$1">
@@
 <wire x1="13.1572" y1="25.8445" x2="13.1572" y2="22.0853" width="0.5588" layer="16"/>
 <wire x1="25.3746" y1="22.5552" x2="25.4" y2="22.86" width="0.5588" layer="16"/>
+<contactref element="BUZZER" pad="-"/>
+<wire x1="4.2291" y1="27.7241" x2="3.81" y2="27.94" width="0" layer="19" extent="16-16"/>
+</signal>
+<signal name="VDD">
+<contactref element="R2" pad="1"/>
+<contactref element="D3" pad="A"/>
+<wire x1="29.1338" y1="50.7492" x2="35.2425" y2="44.6405" width="0.5588" layer="16"/>
+<wire x1="35.2425" y1="44.6405" x2="35.56" y2="44.45" width="0.5588" layer="16"/>
+<wire x1="26.3144" y1="47.9298" x2="15.5067" y2="47.9298" width="0.5588" layer="16"/>
+<wire x1="29.1338" y1="50.7492" x2="26.3144" y2="47.9298" width="0.5588" layer="16"/>
+<wire x1="29.1338" y1="50.7492" x2="29.21" y2="50.8" width="0.5588" layer="16"/>
 </signal>
 </signals>
